File: PCB Design/COMMs_Rev_1/RX.kicad_sch (KiCad schematic)
At the start: 70 parts, among them U10 OPA2322AID, U11 OPA2322AID, U7 INA333AIDGKR, U8 OPA2322AID, U9 AD5246BKSZ50-RL7

Commit message: Small Updates
Other:
- note added: "Should be a 100k ohm resistor"
Changed lines of the file:
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@@
+		)
+	)
+	(text "Should be a 100k ohm resistor"
+		(exclude_from_sim no)
+		(at 53.848 150.368 0)
+		(effects
+			(font
+				(size 1.27 1.27)
+			)
 		)
 	)
