File: PCB Design/COMMs_Rev_2/RX_Rev_2/RX.kicad_pcb (KiCad board)
At the start: 2 copper layers, 40 x 65 mm, 2 parts, among them J1 Conn_01x24_Pin, J2 Conn_01x24_Pin

Commit message: Initial PCB Placement
Parts:
- added C1: 10u, Capacitor_SMD:C_1206_3216Metric, F.Cu at (145.2, 49.8)
- added C10: 100n, Capacitor_SMD:C_0603_1608Metric, F.Cu at (157.5, 94.6)
- added C11: 10n, Capacitor_SMD:C_0603_1608Metric, F.Cu at (153.8, 82.9)
- added C12: 10n, Capacitor_SMD:C_0603_1608Metric, F.Cu at (153.8, 87.1)
- added C13: 4.7n, Capacitor_SMD:C_0603_1608Metric, F.Cu at (155.5, 99.6)
- added C14: 1n, Capacitor_SMD:C_0603_1608Metric, F.Cu at (144.8, 89.2)
- added C2: 100n, Capacitor_SMD:C_0603_1608Metric, F.Cu at (143.0, 49.8)
- added C3: 100n, Capacitor_SMD:C_0603_1608Metric, F.Cu at (163.0, 98.8)
- added C4: 100n, Capacitor_SMD:C_0603_1608Metric, F.Cu at (165.2, 87.8)
- added C5: 100n, Capacitor_SMD:C_0603_1608Metric, F.Cu at (165.4, 82.0)
- added C6: ~, Capacitor_SMD:C_0603_1608Metric, F.Cu at (154.5, 55.9)
- added C7: 1u, Capacitor_SMD:C_0603_1608Metric, F.Cu at (155.2, 82.9)
- added C8: 100n, Capacitor_SMD:C_0603_1608Metric, F.Cu at (157.0, 82.9)
- added C9: 1u, Capacitor_SMD:C_0603_1608Metric, F.Cu at (157.5, 92.9)
- added J3: Conn_01x03_Pin, Connector_PinHeader_2.54mm:PinHeader_1x03_P2.54mm_Vertical, F.Cu at (166.0, 99.8)
- added J4: Conn_01x04_Pin, Connector_PinHeader_2.54mm:PinHeader_1x04_P2.54mm_Vertical, F.Cu at (150.7, 63.6)
- added J5: Conn_01x02_Pin, Connector_JST:JST_VH_B2P-VH_1x02_P3.96mm_Vertical, F.Cu at (152.5, 49.6)
- added R1: 0, Resistor_SMD:R_0603_1608Metric, F.Cu at (146.5, 57.2)
- added R10: 1k, Resistor_SMD:R_0603_1608Metric, F.Cu at (150.8, 60.8)
- added R11: 100, Resistor_SMD:R_0603_1608Metric, F.Cu at (155.5, 60.1)
- added R12: 1k, Resistor_SMD:R_0603_1608Metric, F.Cu at (158.2, 60.8)
- added R13: ~, Resistor_SMD:R_0603_1608Metric, F.Cu at (154.5, 57.6)
- added R14: R_GAIN, Resistor_SMD:R_0603_1608Metric, F.Cu at (158.0, 77.6)
- added R15: 820, Resistor_SMD:R_0603_1608Metric, F.Cu at (152.0, 87.1)
- added R16: 680, Resistor_SMD:R_0603_1608Metric, F.Cu at (153.0, 97.1)
- added R17: 680, Resistor_SMD:R_0603_1608Metric, F.Cu at (153.0, 100.4)
- added R18: 100k, Resistor_SMD:R_0603_1608Metric, F.Cu at (156.2, 87.9)
- added R19: 100k, Resistor_SMD:R_0603_1608Metric, F.Cu at (155.5, 96.4)
- added R2: 100k, Resistor_SMD:R_0603_1608Metric, F.Cu at (166.7, 86.0)
- added R20: 100, Resistor_SMD:R_0603_1608Metric, F.Cu at (145.5, 91.8)
- added R21: 100k, Resistor_SMD:R_0603_1608Metric, F.Cu at (145.5, 93.5)
- added R22: 100k, Resistor_SMD:R_0603_1608Metric, F.Cu at (152.8, 73.4)
- added R23: 100k, Resistor_SMD:R_0603_1608Metric, F.Cu at (156.2, 73.4)
- added R3: 100k, Resistor_SMD:R_0603_1608Metric, F.Cu at (166.7, 84.2)
- added R4: 10, Resistor_SMD:R_0603_1608Metric, F.Cu at (162.7, 88.5)
- added R5: 100, Resistor_SMD:R_0603_1608Metric, F.Cu at (151.8, 67.4)
- added R6: 100, Resistor_SMD:R_0603_1608Metric, F.Cu at (152.8, 70.9)
- added R7: 100, Resistor_SMD:R_0603_1608Metric, F.Cu at (157.2, 67.4)
- added R8: 100, Resistor_SMD:R_0603_1608Metric, F.Cu at (156.2, 70.9)
- added R9: 100, Resistor_SMD:R_0603_1608Metric, F.Cu at (153.5, 60.1)
- added TP1: TestPoint, TestPoint:TestPoint_Pad_1.0x1.0mm, F.Cu at (160.0, 71.2)
- added TP2: TestPoint, TestPoint:TestPoint_Pad_1.0x1.0mm, F.Cu at (149.0, 71.0)
- added TP3: TestPoint, TestPoint:TestPoint_Pad_1.0x1.0mm, F.Cu at (150.2, 79.2)
- added TP4: TestPoint, TestPoint:TestPoint_Pad_1.0x1.0mm, F.Cu at (158.8, 100.0)
- added TP5: TestPoint, TestPoint:TestPoint_Pad_1.0x1.0mm, F.Cu at (148.2, 90.5)
- added U1: TLV9101IDCKR, RX:SC70-5_DCK_TEX, F.Cu at (163.6, 84.9)
- added U2: TPD2E007DCKR, RX:DCK3, F.Cu at (154.5, 67.4)
- added U3: INA828IDR, RX:D0008A_L, F.Cu at (154.5, 77.8)
- added U4: OPA2322AIDGKR, RX:DGK8, F.Cu at (154.0, 92.1)
Connections:
- J1 pad 10: /GPIO_9 -> unconnected-(J1-Pin_10-Pad10)
- J1 pad 11: /GPIO_10 -> unconnected-(J1-Pin_11-Pad11)
- J1 pad 12: /GPIO_11 -> unconnected-(J1-Pin_12-Pad12)
- J1 pad 13: /GPIO_12 -> unconnected-(J1-Pin_13-Pad13)
- J1 pad 14: /GPIO_13 -> unconnected-(J1-Pin_14-Pad14)
- J1 pad 15: /GPIO_14 -> unconnected-(J1-Pin_15-Pad15)
- J1 pad 16: /ADC1_IN0 -> /ADC_OUT
- J1 pad 17: /ADC1_IN1 -> unconnected-(J1-Pin_17-Pad17)
- J1 pad 18: /ADC1_IN2 -> unconnected-(J1-Pin_18-Pad18)
- J1 pad 19: /ADC1_IN3 -> unconnected-(J1-Pin_19-Pad19)
- J1 pad 20: /PC5 -> unconnected-(J1-Pin_20-Pad20)
- J1 pad 21: /PB0 -> unconnected-(J1-Pin_21-Pad21)
- J1 pad 22: /PB1 -> unconnected-(J1-Pin_22-Pad22)
- J1 pad 23: /HI_A -> unconnected-(J1-Pin_23-Pad23)
- J1 pad 24: /LI_A -> unconnected-(J1-Pin_24-Pad24)
- J1 pad 3: 12V -> unconnected-(J1-Pin_3-Pad3)
- J1 pad 5: V_Piezo -> unconnected-(J1-Pin_5-Pad5)
- J1 pad 7: /GPIO_6 -> unconnected-(J1-Pin_7-Pad7)
- J1 pad 8: /GPIO_7 -> unconnected-(J1-Pin_8-Pad8)
- J1 pad 9: /GPIO_8 -> unconnected-(J1-Pin_9-Pad9)
- J2 pad 1: /PC3 -> unconnected-(J2-Pin_1-Pad1)
- J2 pad 10: /PB12 -> unconnected-(J2-Pin_10-Pad10)
- J2 pad 11: /PB14 -> unconnected-(J2-Pin_11-Pad11)
- J2 pad 12: /PB15 -> unconnected-(J2-Pin_12-Pad12)
- J2 pad 13: /PC6 -> unconnected-(J2-Pin_13-Pad13)
- J2 pad 14: /PC7 -> unconnected-(J2-Pin_14-Pad14)
- J2 pad 15: /PC8 -> unconnected-(J2-Pin_15-Pad15)
- J2 pad 16: /PC9 -> unconnected-(J2-Pin_16-Pad16)
- J2 pad 17: /PA9 -> unconnected-(J2-Pin_17-Pad17)
- J2 pad 18: /PA10 -> unconnected-(J2-Pin_18-Pad18)
- J2 pad 19: /SCL -> unconnected-(J2-Pin_19-Pad19)
- J2 pad 2: /PC0 -> unconnected-(J2-Pin_2-Pad2)
- J2 pad 20: /SDA -> unconnected-(J2-Pin_20-Pad20)
- J2 pad 21: /PB6 -> unconnected-(J2-Pin_21-Pad21)
- J2 pad 22: /PB5 -> unconnected-(J2-Pin_22-Pad22)
- J2 pad 23: /HI_B -> unconnected-(J2-Pin_23-Pad23)
- J2 pad 24: /LI_B -> unconnected-(J2-Pin_24-Pad24)
- J2 pad 3: /PC13 -> unconnected-(J2-Pin_3-Pad3)
- J2 pad 4: /GPIO_28 -> unconnected-(J2-Pin_4-Pad4)
- J2 pad 5: /GPIO_27 -> unconnected-(J2-Pin_5-Pad5)
- J2 pad 6: /GPIO_26 -> unconnected-(J2-Pin_6-Pad6)
- J2 pad 7: /GPIO_17 -> unconnected-(J2-Pin_7-Pad7)
- J2 pad 8: /GPIO_16 -> unconnected-(J2-Pin_8-Pad8)
- J2 pad 9: /PC4 -> unconnected-(J2-Pin_9-Pad9)
Routing:
- net 3.3V: track 0.00 -> 78.4 mm, vias 0 -> 3
- net GND: track 0.00 -> 60.7 mm, vias 0 -> 13
- net V_REF_HALF: track 0.00 -> 47.5 mm, vias 0 -> 4
- net /HPF_OUT: track 0.00 -> 22.4 mm
- net /Piezo_P: track 0.00 -> 12.8 mm
- net /Piezo_N: track 0.00 -> 12.8 mm
- net /ADC_OUT: track 0.00 -> 12.7 mm
- net /BPF_OUT: track 0.00 -> 11.2 mm
- net /HYBRID_RX_P: track 0.00 -> 8.52 mm
- net /HYBRID_RX_N: track 0.00 -> 8.52 mm
- net /RX_P: track 0.00 -> 7.93 mm
- net /RX_N: track 0.00 -> 7.82 mm
- net /LNA_OUT: track 0.00 -> 5.96 mm
- net Net-(U1-IN+): track 0.00 -> 5.94 mm
- net Net-(C11-Pad2): track 0.00 -> 4.47 mm
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- added copper zone on B.Cu, net AGND
- added copper zone on F.Cu, net AGND
- added copper zone on B.Cu, net GND
- added copper zone on F.Cu, net GND
Other:
- board text added: "ADC_OUT"
- board text removed: "12V"
- board text removed: "ADC1_IN0"
- board text removed: "ADC1_IN1"
- board text removed: "ADC1_IN2"
- board text removed: "ADC1_IN3"
- board text removed: "B0"
- board text removed: "B1"
- board text removed: "GPIO10"
- board text removed: "GPIO11"
- board text removed: "GPIO12"
- board text removed: "GPIO13"
- board text removed: "GPIO14"
- board text removed: "GPIO16"
- board text removed: "GPIO17"
- board text removed: "GPIO26"
- board text removed: "GPIO27"
- board text removed: "GPIO28"
- board text removed: "GPIO6"
- board text removed: "GPIO7"
- board text removed: "GPIO8"
- board text removed: "GPIO9"
- board text removed: "PA10"
- board text removed: "PA9"
- board text removed: "PB12"
- board text removed: "PB14"
- board text removed: "PB15"
- board text removed: "PB5"
- board text removed: "PB6"
- board text removed: "PC4"
- board text removed: "PC5"
- board text removed: "PC6"
- board text removed: "PC7"
- board text removed: "PC8"
- board text removed: "PC9"
- board text removed: "PG_12"
- board text removed: "PG_3.3"
- board text removed: "PG_VPi"
- board text removed: "SCL"
- board text removed: "SDA"
- board text removed: "V_Pi"

Commit message: Added Title Summary and Updated Rev 2.1
Other:
- board text added: "TX BOARD REV2.1 03/2026 By Samantha Chong"
- board text removed: "TX BOARD REV2 03/2026 By Samantha Chong"
Changed lines of the file:
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@@
 		)
 	)
-	(gr_text "TX BOARD \nREV2 03/2026\nBy Samantha Chong"
+	(gr_text "TX BOARD \nREV2.1 03/2026\nBy Samantha Chong"
 		(at 157.9 108.8 0)
 		(layer "B.SilkS")
