File: PCB Design/COMMs_Rev_2/RX_Rev_2/RX.kicad_pcb (KiCad board)
At the start: 2 copper layers, 40 x 65 mm, 51 parts, among them J1 Conn_01x24_Pin, J2 Conn_01x24_Pin, J3 Conn_01x03_Pin, J4 Conn_01x04_Pin, J5 Conn_01x02_Pin, U1 TLV9101IDCKR, U2 TPD2E007DCKR, U3 INA828IDR, U4 OPA2322AIDGKR

Commit message: Updated RX
Routing:
- net AGND: track 0.00 -> 2.28 mm
Other:
- board text added: "RX BOARD REV2.2 04/2026 By Samantha Chong"
- board text removed: "TX BOARD REV2.1 03/2026 By Samantha Chong"

Commit message: Updated
Routing:
- net AGND: vias 181 -> 183

Commit message: Revert "Updated"
This reverts commit 89be44ed720659141c8ee702c54a520a60db740f.
Routing:
- net AGND: vias 183 -> 181
