File: SWARM_PCB_Rev_2/CONTROL.kicad_sch (KiCad schematic)
At the start: 53 parts, among them J1 Conn_01x02_Pin, J6 USB_C_Receptacle_USB2.0_16P, J7 Micro_SD_Card, J8 Conn_01x06_Pin, U1 STM32F446RET6, U2 USBLC6-2SC6, Y1 32.768KHz, Y2 16MHz

Commit message: Reannotated Schematic
Parts:
- removed D2: MINT, symbol Device:LED
- removed R6: 1k, symbol Device:R_US
- JP1, JP2, JP3: footprint (none) -> Jumper:SolderJumper-2_P1.3mm_Open_TrianglePad1.0x1.5mm
- aC1: renamed from C1; footprint (none) -> Capacitor_SMD:C_0603_1608Metric
- aC10: renamed from C4; footprint (none) -> Capacitor_SMD:C_0603_1608Metric
- aC11: renamed from C5; footprint (none) -> Capacitor_SMD:C_0603_1608Metric
- aC12: renamed from C6; footprint (none) -> Capacitor_SMD:C_0603_1608Metric
- aC13: renamed from C7; footprint (none) -> Capacitor_SMD:C_0603_1608Metric
- aC14: renamed from C8; footprint (none) -> Capacitor_SMD:C_0603_1608Metric
- aC15: renamed from C9; footprint (none) -> Capacitor_SMD:C_0603_1608Metric
- aC16: renamed from C10; footprint (none) -> Capacitor_SMD:C_0603_1608Metric
- aC17: renamed from C11; footprint (none) -> Capacitor_SMD:C_0603_1608Metric
- aC18: renamed from C12; footprint (none) -> Capacitor_SMD:C_0603_1608Metric
- aC19: renamed from C13; footprint (none) -> Capacitor_SMD:C_0603_1608Metric
- aC2: renamed from C17; footprint (none) -> Capacitor_SMD:C_0603_1608Metric
- aC3: renamed from C2; footprint (none) -> Capacitor_SMD:C_0603_1608Metric
- aC4: renamed from C18; footprint (none) -> Capacitor_SMD:C_0603_1608Metric
- aC5: renamed from C19; footprint (none) -> Capacitor_SMD:C_0603_1608Metric
- aC6: renamed from C14; footprint (none) -> Capacitor_SMD:C_0603_1608Metric
- aC7: renamed from C15; footprint (none) -> Capacitor_SMD:C_0603_1608Metric
- aC8: renamed from C16; footprint (none) -> Capacitor_SMD:C_0603_1608Metric
- aC9: renamed from C3; footprint (none) -> Capacitor_SMD:C_0603_1608Metric
- aD1: renamed from D1; footprint (none) -> SWARM_LIBRARY:LED_JE2835_CRW
- aD2: renamed from D3; footprint (none) -> LED_SMD:LED_RGB_PLCC-6
- aFB1: renamed from FB1; footprint (none) -> Resistor_SMD:R_0603_1608Metric
- aJ1: renamed from J1; footprint (none) -> Connector_PinHeader_1.00mm:PinHeader_1x02_P1.00mm_Vertical
- aJ2: renamed from J6; footprint (none) -> Connector_USB:USB_C_Receptacle_GCT_USB4085
- aJ3: renamed from J7; footprint (none) -> SWARM_LIBRARY:AMPHENOL_1140084168
- aJ4: renamed from J8; footprint (none) -> Connector_PinHeader_1.00mm:PinHeader_1x06_P1.00mm_Vertical
- aR1: renamed from R7; footprint (none) -> Resistor_SMD:R_0603_1608Metric
- aR10: renamed from R3; footprint (none) -> Resistor_SMD:R_0603_1608Metric
- aR11: renamed from R4; footprint (none) -> Resistor_SMD:R_0603_1608Metric
- aR12: renamed from R19; footprint (none) -> Resistor_SMD:R_0603_1608Metric
- aR13: renamed from R13; footprint (none) -> Resistor_SMD:R_0603_1608Metric
- aR14: renamed from R14; footprint (none) -> Resistor_SMD:R_0603_1608Metric
- aR15: renamed from R15; footprint (none) -> Resistor_SMD:R_0603_1608Metric
- aR16: renamed from R16; footprint (none) -> Resistor_SMD:R_0603_1608Metric
- aR17: renamed from R17; footprint (none) -> Resistor_SMD:R_0603_1608Metric
- aR2: renamed from R8; footprint (none) -> Resistor_SMD:R_0603_1608Metric
- aR3: renamed from R9; footprint (none) -> Resistor_SMD:R_0603_1608Metric
- aR4: renamed from R5; footprint (none) -> Resistor_SMD:R_0603_1608Metric
- aR5: renamed from R2; footprint (none) -> Resistor_SMD:R_0603_1608Metric
- aR6: renamed from R1; footprint (none) -> Resistor_SMD:R_0603_1608Metric
- aR7: renamed from R11; footprint (none) -> Resistor_SMD:R_0603_1608Metric
- aR8: renamed from R12; footprint (none) -> Resistor_SMD:R_0603_1608Metric
- aR9: renamed from R18; footprint (none) -> Resistor_SMD:R_0603_1608Metric
- aU1: renamed from A1; footprint Module:RaspberryPi_Pico_Common_Unspecified -> Module:RaspberryPi_Pico_SMD
- aY1: renamed from Y1; footprint (none) -> Crystal:Crystal_SMD_MicroCrystal_CM9V-T1A-2Pin_1.6x1.0mm
- aY2: renamed from Y2; footprint (none) -> Crystal:Crystal_SMD_SeikoEpson_FA238-4Pin_3.2x2.5mm
- renumbered U1 to aU2, U2 to aU3
Connections:
- net GND_CONTROL: no longer aU1.33 (AGND)
- net GPIO_15: no longer names the net of aU1.20 (GPIO15)
- net STM_UART_RX: no longer names the net of aU2.52 (PC11)
- net STM_UART_RX: no longer aU1.1 (GPIO0)
- net STM_UART_TX: no longer names the net of aU2.51 (PC10)
- net STM_UART_TX: no longer aU1.2 (GPIO1)
- no-connect marks 4 -> 5
Other:
- note removed: "UART0"
- note removed: "UART4"
- moved on the sheet: aD1, aR4

Commit message: Finished Placement for POWER, CONTROL and SENSOR
Connections:
- net GPIO_16 is gone; now on net SWO_P: aU1.21 (GPIO16)
- net GPIO_17 is gone; now on net NRST_P: aU1.22 (GPIO17)
- net BOOT0_P: now also aU1.26 (GPIO20); no longer aU1.25 (GPIO19)
- net NRST_P: no longer aU1.24 (GPIO18)
- net SWCLK_P: now also aU1.25 (GPIO19); no longer aU1.27 (GPIO21)
- net SWDIO_P: now also aU1.24 (GPIO18); no longer aU1.29 (GPIO22)
- net SWO_P: no longer aU1.26 (GPIO20)
- net PC10: now reaches aU2.51 (PC10)
- net PC11: now reaches aU2.52 (PC11)
- net GPIO_0: now reaches aU1.1 (GPIO0)
- net GPIO_1: now reaches aU1.2 (GPIO1)
- net GPIO_15: now reaches aU1.20 (GPIO15)
- new net GPIO_21: aU1.27 (GPIO21)
- new net GPIO_22: aU1.29 (GPIO22)
Other:
- sheet HEADER_PINS ports: added PIN_1, PIN_10, PIN_11, PIN_12, PIN_13, PIN_14, PIN_15, PIN_16, PIN_17, PIN_18, PIN_19, PIN_2, PIN_20, PIN_21, PIN_22, PIN_23, PIN_24, PIN_25, PIN_26, PIN_27, PIN_28, PIN_29, PIN_3, PIN_30, PIN_31, PIN_32, PIN_33, PIN_34, PIN_35, PIN_36, PIN_37, PIN_38, PIN_39, PIN_4, PIN_40, PIN_41, PIN_42, PIN_43, PIN_44, PIN_45, PIN_46, PIN_47, PIN_5, PIN_6, PIN_7, PIN_8, PIN_9; removed ADC1_IN0, ADC1_IN1, ADC1_IN2, ADC1_IN3, GPIO_10, GPIO_11, GPIO_12, GPIO_13, GPIO_14, GPIO_16, GPIO_17, GPIO_26, GPIO_27, GPIO_28, GPIO_6, GPIO_7, GPIO_8, GPIO_9, HI_A, HI_B, LI_A, LI_B, PA10, PA9, PB0, PB1, PB12, PB14, PB15, PB5, PB6, PC0, PC13, PC3, PC4, PC5, PC6, PC7, PC8, PC9, SCL, SDA
