File: SWARM_PCB_Rev_2/CONTROL.kicad_sch (KiCad schematic)
At the start: 52 parts

Commit message: Fix HSE crystal load cap MPNs and update design review
- CONTROL: aC18/aC19 MPN updated to GRM1885C1H100JA01D (10pF C0G 50V 0603)
  to match corrected Value=10p; was GRM188R61A105KA61D (1uF - wrong part)
- CONTROL: aC16/aC17 1uF decoupling cap MPNs restored (collateral from replace_all)
- DESIGN_REVIEW: close C2, P6, T5; downgrade T4; note piezo load context

Co-Authored-By: Claude Sonnet 4.6 <noreply@anthropic.com>
Parts:
- aC18, aC19: value 1u -> 10p; MPN GRM188R61A105KA61D -> GRM1885C1H100JA01D
Changed lines of the file:
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@@
 			)
 		)
-		(property "Value" "1u"
+		(property "Value" "10p"
 			(at 104.394 184.912 0)
 			(show_name no)
@@
 			)
 		)
-		(property "MPN" "GRM188R61A105KA61D"
+		(property "MPN" "GRM1885C1H100JA01D"
 			(at 0 0 0)
 			(hide yes)
@@
 			)
 		)
-		(property "Value" "1u"
+		(property "Value" "10p"
 			(at 86.614 184.912 0)
 			(show_name no)
@@
 			)
 		)
-		(property "MPN" "GRM188R61A105KA61D"
+		(property "MPN" "GRM1885C1H100JA01D"
 			(at 0 0 0)
 			(hide yes)

Commit message: Fix aC15 decoupling cap 10nF→100nF; close C5 and C6 findings
- aC15: Value 10n→100n, MPN GRM188R71H103KA01D→GRM188R71C104KA01D
  (meets ST ≥100nF recommendation for VBAT/VDD decoupling)
- C5 closed: VBAT confirmed tied to +3.3V_CONTROL
- C6 closed: NRST filter cap aC1 = 100nF confirmed

Co-Authored-By: Claude Sonnet 4.6 <noreply@anthropic.com>
Parts:
- aC15: value 10n -> 100n; MPN GRM188R71H103KA01D -> GRM188R71C104KA01D
Changed lines of the file:
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@@
 			)
 		)
-		(property "Value" "10n"
+		(property "Value" "100n"
 			(at 26.924 177.292 0)
 			(show_name no)
@@
 			)
 		)
-		(property "MPN" "GRM188R71H103KA01D"
+		(property "MPN" "GRM188R71C104KA01D"
 			(at 0 0 0)
 			(hide yes)
