File: SWARM_PCB_Rev_2/CONTROL.kicad_sch (KiCad schematic)
At the start: 52 parts

Commit message: Fixed some small errors and added the Output board
Parts:
- aR10, aR11: value 4.7k -> 2.2k
Connections:
- net SWCLK: no longer aR18.1
- net at JP1.1 (A): now also aR18.1
Changed lines of the file:
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@@
 	(wire
 		(pts
-			(xy 173.99 110.49) (xy 185.42 110.49)
-		)
-		(stroke
-			(width 0)
-			(type default)
-		)
-	)
-	(wire
-		(pts
 			(xy 116.84 114.3) (xy 116.84 111.76)
 		)
@@
 	(wire
 		(pts
+			(xy 173.99 110.49) (xy 175.26 110.49)
+		)
+		(stroke
+			(width 0)
+			(type default)
+		)
+	)
+	(wire
+		(pts
 			(xy 130.81 146.05) (xy 138.43 146.05)
 		)
@@
 			)
 		)
-		(property "Value" "4.7k"
+		(property "Value" "2.2k"
 			(at 117.094 121.158 0)
 			(show_name no)
@@
 			)
 		)
-		(property "Value" "4.7k"
+		(property "Value" "2.2k"
 			(at 109.474 121.158 0)
 			(show_name no)
