File: SWARM_PCB_Rev_2/CONTROL.kicad_sch (KiCad schematic)
At the start: 53 parts

Commit message: Updated Via size to 0.25mm and ReExported Files
Parts:
- aC1, aC10, aC11, aC12, aC13, aC14, aC15, aC16, aC17, aC18, aC19, aC2, aC3, aC4, aC5, aC6, aC7, aC8, aC9, aFB1: Manufacturer Murata -> (none)
- aJ2: Manufacturer GCT -> (none)
- aJ3: Manufacturer Amphenol -> (none)
- aR1, aR10, aR11, aR12, aR13, aR14, aR15, aR16, aR17, aR18, aR19, aR2, aR3, aR4, aR5, aR6, aR7, aR8, aR9: Manufacturer Yageo -> (none)
- aU1: Manufacturer Raspberry Pi -> (none)
- aU2, aU3: Manufacturer STMicroelectronics -> (none)
- aY1: Manufacturer MicroCrystal -> (none)
- aY2: Manufacturer Seiko Epson -> (none)

Commit message: Cleaned up Schematic and Exported
Other:
- moved on the sheet: aC6, aC7, aC8, aJ4
