File: SWARM_PCB_Rev_2/SENSOR.kicad_sch (KiCad schematic)
At the start: 14 parts, among them U3 MS583730BA01-50, U4 ASM330LHHXTR, U5 LSM6DSO32TR, U6 MMC5603NJ

Commit message: Reannotated Schematic
Parts:
- cC1: renamed from C21; footprint (none) -> Capacitor_SMD:C_0603_1608Metric
- cC2: renamed from C25; footprint (none) -> Capacitor_SMD:C_0603_1608Metric
- cC3: renamed from C26; footprint (none) -> Capacitor_SMD:C_0603_1608Metric
- cC4: renamed from C27; footprint (none) -> Capacitor_SMD:C_0603_1608Metric
- cC5: renamed from C20; footprint (none) -> Capacitor_SMD:C_0603_1608Metric
- cC6: renamed from C22; footprint (none) -> Capacitor_SMD:C_0603_1608Metric
- cC7: renamed from C23; footprint (none) -> Capacitor_SMD:C_0603_1608Metric
- cC8: renamed from C24; footprint (none) -> Capacitor_SMD:C_0603_1608Metric
- cR1: renamed from R10; footprint (none) -> Resistor_SMD:R_0603_1608Metric
- cR2: renamed from R20; footprint (none) -> Resistor_SMD:R_0603_1608Metric
- cU1: renamed from U6; Availability In Stock -> (none); Package UFBGA-4 Memsic Inc. -> (none); Price None -> (none)
- cU2: renamed from U4; Availability In Stock -> (none); Package VFLGA-14 STMicroelectronics -> (none); Price None -> (none)
- cU4: renamed from U5; Availability In Stock -> (none); Package VFLGA-14 STMicroelectronics -> (none); Price None -> (none)
- renumbered U3 to cU3

Commit message: Finished Placement for POWER, CONTROL and SENSOR
Connections:
- no-connect marks 37 -> 46
Other:
- sheet HEADER_PINS ports: added PIN_1, PIN_10, PIN_11, PIN_12, PIN_13, PIN_14, PIN_15, PIN_16, PIN_17, PIN_18, PIN_19, PIN_2, PIN_20, PIN_21, PIN_22, PIN_23, PIN_24, PIN_25, PIN_26, PIN_27, PIN_28, PIN_29, PIN_3, PIN_30, PIN_31, PIN_32, PIN_33, PIN_34, PIN_35, PIN_36, PIN_37, PIN_38, PIN_39, PIN_4, PIN_40, PIN_41, PIN_42, PIN_43, PIN_44, PIN_45, PIN_46, PIN_47, PIN_5, PIN_6, PIN_7, PIN_8, PIN_9; removed ADC1_IN0, ADC1_IN1, ADC1_IN2, ADC1_IN3, GPIO_10, GPIO_11, GPIO_12, GPIO_13, GPIO_14, GPIO_16, GPIO_17, GPIO_26, GPIO_27, GPIO_28, GPIO_6, GPIO_7, GPIO_8, GPIO_9, HI_A, HI_B, LI_A, LI_B, PA10, PA9, PB0, PB1, PB12, PB14, PB15, PB5, PB6, PC0, PC13, PC3, PC4, PC5, PC6, PC7, PC8, PC9, SCL, SDA
- note added: "Address:0x30"
- note added: "Address:0x76"
- note removed: "Address:"

Commit message: Completed PCB Layout
Parts:
- cU4: Availability (none) -> In Stock; Package (none) -> VFLGA-14 STMicroelectronics; Price (none) -> None
Connections:
- no-connect marks 46 -> 42
Changed lines of the file:
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@@
 	(paper "A4")
 	(title_block
-		(date "2026-05-26")
+		(date "2026-05-27")
 		(company "ASTRELIS NAV")
 		(comment 1 "By SAMANTHA CHONG")
@@
 	(rectangle
 		(start 187.96 12.7)
-		(end 217.17 33.02)
+		(end 210.82 33.02)
 		(stroke
 			(width 0.254)
@@
 	)
 	(no_connect
-		(at 270.51 67.31)
-	)
-	(no_connect
 		(at 247.65 41.91)
 	)
@@
 	)
 	(no_connect
-		(at 270.51 74.93)
-	)
-	(no_connect
 		(at 247.65 72.39)
 	)
@@
 	)
 	(no_connect
-		(at 270.51 69.85)
-	)
-	(no_connect
 		(at 270.51 34.29)
 	)
@@
 	)
 	(no_connect
-		(at 270.51 64.77)
-	)
-	(no_connect
 		(at 247.65 54.61)
 	)
@@
 	(wire
 		(pts
+			(xy 270.51 64.77) (xy 283.21 64.77)
+		)
+		(stroke
+			(width 0)
+			(type default)
+		)
+	)
+	(wire
+		(pts
 			(xy 246.38 26.67) (xy 247.65 26.67)
 		)
@@
 	(wire
 		(pts
-			(xy 193.04 24.13) (xy 193.04 26.67)
+			(xy 194.31 24.13) (xy 194.31 26.67)
 		)
 		(stroke
@@
 	(wire
 		(pts
+			(xy 270.51 69.85) (xy 283.21 69.85)
+		)
+		(stroke
+			(width 0)
+			(type default)
+		)
+	)
+	(wire
+		(pts
 			(xy 16.51 33.02) (xy 16.51 39.37)
 		)
@@
 	(wire
 		(pts
+			(xy 270.51 74.93) (xy 283.21 74.93)
+		)
+		(stroke
+			(width 0)
+			(type default)
+		)
+	)
+	(wire
+		(pts
 			(xy 90.17 26.67) (xy 90.17 29.21)
 		)
@@
 	(wire
 		(pts
+			(xy 270.51 67.31) (xy 283.21 67.31)
+		)
+		(stroke
+			(width 0)
+			(type default)
+		)
+	)
+	(wire
+		(pts
 			(xy 64.77 45.72) (xy 67.31 45.72)
 		)
@@
 	(wire
 		(pts
-			(xy 203.2 24.13) (xy 203.2 26.67)
+			(xy 204.47 24.13) (xy 204.47 26.67)
 		)
 		(stroke
@@
 		)
 	)
+	(label "ACC2_INT2"
+		(at 283.21 74.93 180)
+		(effects
+			(font
+				(size 1.27 1.27)
+			)
+			(justify right bottom)
+		)
+	)
 	(label "SCL"
 		(at 24.13 38.1 0)
@@
 		)
 	)
+	(label "ACC1_INT1"
+		(at 283.21 64.77 180)
+		(effects
+			(font
+				(size 1.27 1.27)
+			)
+			(justify right bottom)
+		)
+	)
 	(label "ACC2_INT1"
 		(at 15.24 71.12 0)
@@
 		)
 	)
+	(label "ACC2_INT1"
+		(at 283.21 69.85 180)
+		(effects
+			(font
+				(size 1.27 1.27)
+			)
+			(justify right bottom)
+		)
+	)
+	(label "ACC1_INT2"
+		(at 283.21 67.31 180)
+		(effects
+			(font
+				(size 1.27 1.27)
+			)
+			(justify right bottom)
+		)
+	)
 	(label "SDA"
 		(at 67.31 78.74 180)
@@
 	(symbol
 		(lib_id "power:+3.3V")
-		(at 193.04 24.13 0)
+		(at 194.31 24.13 0)
 		(unit 1)
 		(body_style 1)
@@
 		(dnp no)
 		(property "Reference" "#PWR0134"
-			(at 193.04 27.94 0)
+			(at 194.31 27.94 0)
 			(hide yes)
 			(show_name no)
@@
 		)
 		(property "Value" "+3.3V_SENSOR"
-			(at 193.04 20.828 0)
+			(at 194.31 20.828 0)
 			(show_name no)
 			(do_not_autoplace no)
@@
 		)
 		(property "Footprint" ""
-			(at 193.04 24.13 0)
+			(at 194.31 24.13 0)
 			(hide yes)
 			(show_name no)
@@
 		)
 		(property "Datasheet" ""
-			(at 193.04 24.13 0)
+			(at 194.31 24.13 0)
 			(hide yes)
 			(show_name no)
@@
 		)
 		(property "Description" "Power symbol creates a global label with name \"+3.3V\""
-			(at 193.04 24.13 0)
+			(at 194.31 24.13 0)
 			(hide yes)
 			(show_name no)
@@
 	(symbol
 		(lib_id "power:PWR_FLAG")
-		(at 193.04 26.67 180)
+		(at 194.31 26.67 180)
 		(unit 1)
 		(body_style 1)
@@
 		(fields_autoplaced yes)
 		(property "Reference" "#FLG010"
-			(at 193.04 28.575 0)
+			(at 194.31 28.575 0)
 			(hide yes)
 			(show_name no)
@@
 		)
 		(property "Value" "PWR_FLAG"
-			(at 193.04 31.75 0)
+			(at 194.31 31.75 0)
 			(hide yes)
 			(show_name no)
@@
 		)
 		(property "Footprint" ""
-			(at 193.04 26.67 0)
+			(at 194.31 26.67 0)
 			(hide yes)
 			(show_name no)
@@
 		)
 		(property "Datasheet" ""
-			(at 193.04 26.67 0)
+			(at 194.31 26.67 0)
 			(hide yes)
 			(show_name no)
@@
 		)
 		(property "Description" "Special symbol for telling ERC where power comes from"
-			(at 193.04 26.67 0)
+			(at 194.31 26.67 0)
 			(hide yes)
 			(show_name no)
@@
 	(symbol
 		(lib_id "power:PWR_FLAG")
-		(at 203.2 24.13 0)
+		(at 204.47 24.13 0)
 		(unit 1)
 		(body_style 1)
@@
 		(fields_autoplaced yes)
 		(property "Reference" "#FLG09"
-			(at 203.2 22.225 0)
+			(at 204.47 22.225 0)
 			(hide yes)
 			(show_name no)
@@
 		)
 		(property "Value" "PWR_FLAG"
-			(at 203.2 19.05 0)
+			(at 204.47 19.05 0)
 			(hide yes)
 			(show_name no)
@@
 		)
 		(property "Footprint" ""
-			(at 203.2 24.13 0)
+			(at 204.47 24.13 0)
 			(hide yes)
 			(show_name no)
@@
 		)
 		(property "Datasheet" ""
-			(at 203.2 24.13 0)
+			(at 204.47 24.13 0)
 			(hide yes)
 			(show_name no)
@@
 		)
 		(property "Description" "Special symbol for telling ERC where power comes from"
-			(at 203.2 24.13 0)
+			(at 204.47 24.13 0)
 			(hide yes)
 			(show_name no)
@@
 			)
 		)
+		(property "Package" "VFLGA-14 STMicroelectronics"
+			(at 43.18 76.2 0)
+			(hide yes)
+			(show_name no)
+			(do_not_autoplace no)
+			(effects
+				(font
+					(size 1.27 1.27)
+				)
+				(justify bottom)
+			)
+		)
+		(property "Price" "None"
+			(at 43.18 76.2 0)
+			(hide yes)
+			(show_name no)
+			(do_not_autoplace no)
+			(effects
+				(font
+					(size 1.27 1.27)
+				)
+				(justify bottom)
+			)
+		)
+		(property "Availability" "In Stock"
+			(at 43.18 76.2 0)
+			(hide yes)
+			(show_name no)
+			(do_not_autoplace no)
+			(effects
+				(font
+					(size 1.27 1.27)
+				)
+				(justify bottom)
+			)
+		)
 		(pin "6"
 		)
@@
 	(symbol
 		(lib_id "power:GND")
-		(at 203.2 26.67 0)
+		(at 204.47 26.67 0)
 		(unit 1)
 		(body_style 1)
@@
 		(dnp no)
 		(property "Reference" "#PWR0138"
-			(at 203.2 33.02 0)
+			(at 204.47 33.02 0)
 			(hide yes)
 			(show_name no)
@@
 		)
 		(property "Value" "GND_SENSOR"
-			(at 203.2 29.972 0)
+			(at 204.47 29.972 0)
 			(show_name no)
 			(do_not_autoplace no)
@@
 		)
 		(property "Footprint" ""
-			(at 203.2 26.67 0)
+			(at 204.47 26.67 0)
 			(hide yes)
 			(show_name no)
@@
 		)
 		(property "Datasheet" ""
-			(at 203.2 26.67 0)
+			(at 204.47 26.67 0)
 			(hide yes)
 			(show_name no)
@@
 		)
 		(property "Description" "Power symbol creates a global label with name \"GND\" , ground"
-			(at 203.2 26.67 0)
+			(at 204.47 26.67 0)
 			(hide yes)
 			(show_name no)
