File: SWARM_PCB_Rev_2/SENSOR.kicad_sch (KiCad schematic)
At the start: 14 parts

Commit message: Add MPNs to BOM and apply PCB DFM fixes for JLCPCB
Schematic: added MPN and Manufacturer properties to 205 references
across all sub-sheets (Murata/Yageo/TI/ST/Hirose/JST etc.).
Fixed dU7 description to match INA823DR (not INA828).

PCB: added via tenting (1540 vias), removed stale auto-placement-area
keepout zones (4 zones), increased annular rings on 482 undersized vias
(0.05mm -> 0.1mm), added 6 fiducial markers (3x F.Cu + 3x B.Cu).

Co-Authored-By: Claude Sonnet 4.6 <noreply@anthropic.com>
Parts:
- cC1: MPN (none) -> GRM188R60J225KE15D; Manufacturer (none) -> Murata
- cC2, cC3, cC5, cC6, cC7: MPN (none) -> GRM188R71C104KA01D; Manufacturer (none) -> Murata
- cC4, cC8: MPN (none) -> GRM188R60J106ME47D; Manufacturer (none) -> Murata
- cR1, cR2: MPN (none) -> RC0603FR-074K7L; Manufacturer (none) -> Yageo
- cU1: MPN (none) -> MMC5603NJ; Manufacturer (none) -> MEMSIC
- cU2: MPN (none) -> ASM330LHHXTR; Manufacturer (none) -> STMicroelectronics
- cU3: MPN (none) -> MS583730BA01-50; Manufacturer (none) -> TE Connectivity
- cU4: MPN (none) -> LSM6DSO32TR; Manufacturer (none) -> STMicroelectronics
Changed lines of the file:
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@@
 			)
 		)
+		(property "Manufacturer" "MEMSIC" (at 0 0 0)
+			(effects
+				(font
+					(size 1.27 1.27)
+				)
+				(hide yes)
+			)
+		)
+		(property "MPN" "MMC5603NJ" (at 0 0 0)
+			(effects
+				(font
+					(size 1.27 1.27)
+				)
+				(hide yes)
+			)
+		)
 		(pin "A1"
 		)
@@
 			)
 		)
+		(property "Manufacturer" "Murata" (at 0 0 0)
+			(effects
+				(font
+					(size 1.27 1.27)
+				)
+				(hide yes)
+			)
+		)
+		(property "MPN" "GRM188R71C104KA01D" (at 0 0 0)
+			(effects
+				(font
+					(size 1.27 1.27)
+				)
+				(hide yes)
+			)
+		)
 		(pin "2"
 		)
@@
 			)
 		)
+		(property "Manufacturer" "Yageo" (at 0 0 0)
+			(effects
+				(font
+					(size 1.27 1.27)
+				)
+				(hide yes)
+			)
+		)
+		(property "MPN" "RC0603FR-074K7L" (at 0 0 0)
+			(effects
+				(font
+					(size 1.27 1.27)
+				)
+				(hide yes)
+			)
+		)
 		(pin "2"
 		)
@@
 			)
 		)
+		(property "Manufacturer" "STMicroelectronics" (at 0 0 0)
+			(effects
+				(font
+					(size 1.27 1.27)
+				)
+				(hide yes)
+			)
+		)
+		(property "MPN" "ASM330LHHXTR" (at 0 0 0)
+			(effects
+				(font
+					(size 1.27 1.27)
+				)
+				(hide yes)
+			)
+		)
 		(pin "8"
 		)
@@
 			)
 		)
+		(property "Manufacturer" "STMicroelectronics" (at 0 0 0)
+			(effects
+				(font
+					(size 1.27 1.27)
+				)
+				(hide yes)
+			)
+		)
+		(property "MPN" "LSM6DSO32TR" (at 0 0 0)
+			(effects
+				(font
+					(size 1.27 1.27)
+				)
+				(hide yes)
+			)
+		)
 		(pin "6"
 		)
@@
 			)
 		)
+		(property "Manufacturer" "Murata" (at 0 0 0)
+			(effects
+				(font
+					(size 1.27 1.27)
+				)
+				(hide yes)
+			)
+		)
+		(property "MPN" "GRM188R71C104KA01D" (at 0 0 0)
+			(effects
+				(font
+					(size 1.27 1.27)
+				)
+				(hide yes)
+			)
+		)
 		(pin "2"
 		)
@@
 			)
 		)
+		(property "Manufacturer" "Murata" (at 0 0 0)
+			(effects
+				(font
+					(size 1.27 1.27)
+				)
+				(hide yes)
+			)
+		)
+		(property "MPN" "GRM188R60J225KE15D" (at 0 0 0)
+			(effects
+				(font
+					(size 1.27 1.27)
+				)
+				(hide yes)
+			)
+		)
 		(pin "2"
 		)
@@
 			)
 		)
+		(property "Manufacturer" "Murata" (at 0 0 0)
+			(effects
+				(font
+					(size 1.27 1.27)
+				)
+				(hide yes)
+			)
+		)
+		(property "MPN" "GRM188R60J106ME47D" (at 0 0 0)
+			(effects
+				(font
+					(size 1.27 1.27)
+				)
+				(hide yes)
+			)
+		)
 		(pin "2"
 		)
@@
 			)
 		)
+		(property "Manufacturer" "Murata" (at 0 0 0)
+			(effects
+				(font
+					(size 1.27 1.27)
+				)
+				(hide yes)
+			)
+		)
+		(property "MPN" "GRM188R71C104KA01D" (at 0 0 0)
+			(effects
+				(font
+					(size 1.27 1.27)
+				)
+				(hide yes)
+			)
+		)
 		(pin "2"
 		)
@@
 			)
 		)
+		(property "Manufacturer" "Murata" (at 0 0 0)
+			(effects
+				(font
+					(size 1.27 1.27)
+				)
+				(hide yes)
+			)
+		)
+		(property "MPN" "GRM188R60J106ME47D" (at 0 0 0)
+			(effects
+				(font
+					(size 1.27 1.27)
+				)
+				(hide yes)
+			)
+		)
 		(pin "2"
 		)
@@
 			)
 		)
+		(property "Manufacturer" "Murata" (at 0 0 0)
+			(effects
+				(font
+					(size 1.27 1.27)
+				)
+				(hide yes)
+			)
+		)
+		(property "MPN" "GRM188R71C104KA01D" (at 0 0 0)
+			(effects
+				(font
+					(size 1.27 1.27)
+				)
+				(hide yes)
+			)
+		)
 		(pin "2"
 		)
@@
 			)
 		)
+		(property "Manufacturer" "Yageo" (at 0 0 0)
+			(effects
+				(font
+					(size 1.27 1.27)
+				)
+				(hide yes)
+			)
+		)
+		(property "MPN" "RC0603FR-074K7L" (at 0 0 0)
+			(effects
+				(font
+					(size 1.27 1.27)
+				)
+				(hide yes)
+			)
+		)
 		(pin "2"
 		)
@@
 			)
 		)
+		(property "Manufacturer" "Murata" (at 0 0 0)
+			(effects
+				(font
+					(size 1.27 1.27)
+				)
+				(hide yes)
+			)
+		)
+		(property "MPN" "GRM188R71C104KA01D" (at 0 0 0)
+			(effects
+				(font
+					(size 1.27 1.27)
+				)
+				(hide yes)
+			)
+		)
 		(pin "2"
 		)
@@
 			)
 		)
+		(property "Manufacturer" "TE Connectivity" (at 0 0 0)
+			(effects
+				(font
+					(size 1.27 1.27)
+				)
+				(hide yes)
+			)
+		)
+		(property "MPN" "MS583730BA01-50" (at 0 0 0)
+			(effects
+				(font
+					(size 1.27 1.27)
+				)
+				(hide yes)
+			)
+		)

Commit message: Fix VCAP cap value and I2C pull-up resistors
- CONTROL: aC3 VCAP changed 2.2uF -> 1uF (GRM188R60J105KE15D) per STM32F446 spec
- SENSOR: cR1/cR2 I2C pull-ups changed 4.7k -> 2.2k (RC0603FR-072K2L) for 400kHz 4-device bus

Co-Authored-By: Claude Sonnet 4.6 <noreply@anthropic.com>
Parts:
- cR1, cR2: value 4.7k -> 2.2k; MPN RC0603FR-074K7L -> RC0603FR-072K2L
Changed lines of the file:
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@@
 			)
 		)
-		(property "Value" "4.7k"
+		(property "Value" "2.2k"
 			(at 174.244 28.448 0)
 			(show_name no)
@@
 			)
 		)
-		(property "MPN" "RC0603FR-074K7L"
+		(property "MPN" "RC0603FR-072K2L"
 			(at 0 0 0)
 			(hide yes)
@@
 			)
 		)
-		(property "Value" "4.7k"
+		(property "Value" "2.2k"
 			(at 181.864 28.448 0)
 			(show_name no)
@@
 			)
 		)
-		(property "MPN" "RC0603FR-074K7L"
+		(property "MPN" "RC0603FR-072K2L"
 			(at 0 0 0)
 			(hide yes)
