File: SWARM_PCB_Rev_2/SWARM_PCB_Rev_2.kicad_sch (KiCad schematic)
At the start: 0 parts

Commit message: TX Board Schematic
Parts:
- added J25, J26, J27: Conn_01x12_Pin, Connector_PinSocket_2.54mm:PinSocket_1x12_P2.54mm_Vertical, symbol Connector:Conn_01x12_Pin
- added J28: Conn_01x13_Pin, Connector_PinSocket_2.54mm:PinSocket_1x13_P2.54mm_Vertical, symbol Connector:Conn_01x13_Pin
Connections:
- new net +3.3V_HEADER: J25.1 (Pin_1)
- new net ADC1_IN0: J28.12 (Pin_12)
- new net ADC1_IN1: J27.12 (Pin_12)
- new net ADC1_IN2: J28.13 (Pin_13)
- new net ADC1_IN3: J28.10 (Pin_10)
- new net GND_HEADER: J26.1 (Pin_1)
- new net GPIO_0: J28.1 (Pin_1)
- new net GPIO_1: J27.1 (Pin_1)
- new net GPIO_10: J28.4 (Pin_4)
- new net GPIO_11: J27.4 (Pin_4)
- new net GPIO_12: J28.5 (Pin_5)
- new net GPIO_13: J27.5 (Pin_5)
- new net GPIO_14: J28.6 (Pin_6)
- new net GPIO_15: J27.6 (Pin_6)
- new net GPIO_21: J25.10 (Pin_10)
- new net GPIO_22: J26.3 (Pin_3)
- new net GPIO_26: J25.3 (Pin_3)
- new net GPIO_27: J26.2 (Pin_2)
- new net GPIO_28: J25.2 (Pin_2)
- new net GPIO_6: J28.2 (Pin_2)
- new net GPIO_7: J27.2 (Pin_2)
- new net GPIO_8: J28.3 (Pin_3)
- new net GPIO_9: J27.3 (Pin_3)
- new net HI_A: J27.7 (Pin_7)
- new net HI_B: J26.12 (Pin_12)
- new net LI_A: J28.7 (Pin_7)
- new net LI_B: J26.8 (Pin_8)
- new net PA10: J25.8 (Pin_8)
- new net PA9: J26.7 (Pin_7)
- new net PB0: J27.8 (Pin_8)
- new net PB1: J28.8 (Pin_8)
- new net PB12: J25.4 (Pin_4)
- new net PB14: J26.4 (Pin_4)
- new net PB15: J25.5 (Pin_5)
- new net PB5: J26.10 (Pin_10)
- new net PB6: J25.11 (Pin_11)
- new net PC0: J28.11 (Pin_11)
- new net PC10: J25.9 (Pin_9)
- new net PC11: J26.9 (Pin_9)
- new net PC13: J27.10 (Pin_10)
- new net PC3: J27.11 (Pin_11)
- new net PC4: J27.9 (Pin_9)
- new net PC5: J28.9 (Pin_9)
- new net PC6: J26.5 (Pin_5)
- new net PC7: J25.6 (Pin_6)
- new net PC8: J26.6 (Pin_6)
- new net PC9: J25.7 (Pin_7)
- new net SCL: J25.12 (Pin_12)
- new net SDA: J26.11 (Pin_11)
Other:
- added sheet HEADER_PINS (HEADER_PINS.kicad_sch)
- added sheet RX (RX.kicad_sch)
- added sheet TX (TX.kicad_sch)
- note added: "BOARD BREAKOUTS"
- note added: "DUPLICATE FOOTPRINTS BETWEEN BOARDS"
- note added: "HEADER PINS"
- note added: "for testing"
- note added: "stacking connections between boards"

Commit message: Completed PCB Layout
Connections:
- net ADC1_IN2 renamed BPF_OUT
- net ADC1_IN3 renamed ADC_CURRENT
- net PB0 renamed ACC1_INT1
- net PB1 renamed PG_VPiezo
- net PB12 renamed PG_12V
- net PB6 renamed PG_3.3V
- net PC0 renamed RX_FAULT
- net PC13 renamed ACC2_INT2
- net PC3 renamed RX_EN
- net PC4 renamed ACC2_INT1
- net PC5 renamed ACC1_INT2
Other:
- sheet RX renamed TX_RX
- removed sheet TX
- sheet TX_RX: file RX.kicad_sch -> TX_RX.kicad_sch
- note added: "PWR FLAGS"
- moved on the sheet: J25, J26, J27, J28
