File: SWARM_PCB_Rev_2/SWARM_PCB_Rev_2.kicad_sch (KiCad schematic)
At the start: 4 parts, among them J25 Conn_01x12_Pin, J26 Conn_01x12_Pin, J27 Conn_01x12_Pin, J28 Conn_01x13_Pin

Commit message: Fixed some small errors and added the Output board
Connections:
- net PA10 renamed PG_5V
Other:
- added sheet OUTPUT (OUTPUT.kicad_sch)
Changed lines of the file:
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@@
 	(rectangle
 		(start 64.77 13.97)
-		(end 148.59 57.15)
+		(end 149.86 57.15)
 		(stroke
 			(width 0.254)
@@
 	(text "GND DOMAIN ARCHITECTURE\nEach subsystem has an isolated GND domain: GND_POWER, GND_CONTROL,\nGND_SENSOR, GND_TXRX, GND_HEADER. These domains are connected\nthrough the stacking connector pins (J25-J28). No single star point."
 		(exclude_from_sim no)
-		(at 82.55 62.23 0)
+		(at 89.408 62.484 0)
 		(effects
 			(font
@@
 		)
 	)
+	(label "PG_5V"
+		(at 16.51 68.58 0)
+		(effects
+			(font
+				(size 1.27 1.27)
+			)
+			(justify left bottom)
+		)
+	)
 	(label "SCL"
 		(at 67.31 53.34 0)
@@
 		)
 	)
-	(label "PA10"
+	(label "PG_5V"
 		(at 67.31 43.18 0)
 		(effects
@@
 		)
 	)
-	(label "PA10"
-		(at 16.51 68.58 0)
-		(effects
-			(font
-				(size 1.27 1.27)
-			)
-			(justify left bottom)
-		)
-	)
 	(label "PB14"
 		(at 104.14 33.02 180)
@@
 				)
 			)
+		)
+	)
+	(sheet
+		(at 100.33 123.19)
+		(size 66.04 31.75)
+		(exclude_from_sim no)
+		(in_bom yes)
+		(on_board yes)
+		(dnp no)
+		(fields_autoplaced yes)
+		(stroke
+			(width 0.1524)
+			(type solid)
+		)
+		(fill
+			(color 0 0 0 0)
+		)
+		(property "Sheetname" "OUTPUT"
+			(at 100.33 122.4784 0)
+			(show_name no)
+			(do_not_autoplace no)
+			(effects
+				(font
+					(size 1.27 1.27)
+				)
+				(justify left bottom)
+			)
+		)
+		(property "Sheetfile" "OUTPUT.kicad_sch"
+			(at 100.33 155.5246 0)
+			(hide yes)
+			(show_name no)
+			(do_not_autoplace no)
+			(effects
+				(font
+					(size 1.27 1.27)
+				)
+				(justify left top)
+			)
+		)
+		(instances
+			(project "SWARM_PCB_Rev_2"
+				(path "/d61c6b76-225f-4e7b-954b-419fd350b2a8"
+					(page "8")
+				)
+			)

Commit message: Resolved all DRC and ERC errors
Changed lines of the file:
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@@
 	(title_block
 		(title "SWARM PCB")
-		(date "2026-05-27")
+		(date "2026-06-19")
 		(rev "2")
 		(company "ASTRELIS NAV")
@@
 	(sheet
 		(at 210.82 17.78)
-		(size 69.85 40.64)
+		(size 69.85 25.4)
 		(exclude_from_sim no)
 		(in_bom yes)
@@
 		)
 		(property "Sheetfile" "CONTROL.kicad_sch"
-			(at 210.82 59.0046 0)
+			(at 210.82 43.7646 0)
 			(hide yes)
 			(show_name no)
@@
 	)
 	(sheet
-		(at 210.82 128.27)
-		(size 69.85 33.02)
+		(at 210.82 107.95)
+		(size 69.85 24.13)
 		(exclude_from_sim no)
 		(in_bom yes)
@@
 		)
 		(property "Sheetname" "TX_RX"
-			(at 210.82 127.5584 0)
+			(at 210.82 107.2384 0)
 			(show_name no)
 			(do_not_autoplace no)
@@
 		)
 		(property "Sheetfile" "TX_RX.kicad_sch"
-			(at 210.82 161.8746 0)
+			(at 210.82 132.6646 0)
 			(hide yes)
 			(show_name no)
@@
 	)
 	(sheet
-		(at 210.82 66.04)
-		(size 71.12 24.13)
+		(at 210.82 48.26)
+		(size 69.85 24.13)
 		(exclude_from_sim no)
 		(in_bom yes)
@@
 		)
 		(property "Sheetname" "POWER"
-			(at 210.82 65.3284 0)
+			(at 210.82 47.5484 0)
 			(show_name no)
 			(do_not_autoplace no)
@@
 		)
 		(property "Sheetfile" "POWER.kicad_sch"
-			(at 210.82 90.7546 0)
+			(at 210.82 72.9746 0)
 			(hide yes)
 			(show_name no)
@@
 	)
 	(sheet
-		(at 210.82 97.79)
-		(size 71.12 25.4)
+		(at 210.82 77.47)
+		(size 69.85 25.4)
 		(exclude_from_sim no)
 		(in_bom yes)
@@
 		)
 		(property "Sheetname" "SENSOR"
-			(at 210.82 97.0784 0)
+			(at 210.82 76.7584 0)
 			(show_name no)
 			(do_not_autoplace no)
@@
 		)
 		(property "Sheetfile" "SENSOR.kicad_sch"
-			(at 210.82 123.7746 0)
+			(at 210.82 103.4546 0)
 			(hide yes)
 			(show_name no)
@@
 	)
 	(sheet
-		(at 100.33 123.19)
-		(size 66.04 31.75)
+		(at 210.82 137.16)
+		(size 69.85 24.13)
 		(exclude_from_sim no)
 		(in_bom yes)
@@
 		)
 		(property "Sheetname" "OUTPUT"
-			(at 100.33 122.4784 0)
+			(at 210.82 136.4484 0)
 			(show_name no)
 			(do_not_autoplace no)
@@
 		)
 		(property "Sheetfile" "OUTPUT.kicad_sch"
-			(at 100.33 155.5246 0)
+			(at 210.82 161.8746 0)
 			(hide yes)
 			(show_name no)

Commit message: Cleaned up Schematic and Exported
Other:
- note added: "CONTROL — System brain STM32F446RET6 + Raspberry Pi Pico 2 run main flight logic and higher-level processing. Includes USB-C input (with ESD protection), microSD logging, SWD programming header, RGB/status LEDs, 16MHz/32.768kHz crystals, and a boot-mode jumper for the Pico."
- note added: "GND DOMAIN ARCHITECTURE Each subsystem has an isolated GND domain: GND_POWER, GND_CONTROL, GND_SENSOR, GND_TXRX, GND_HEADER. These domains are connected through the stacking connector pins. No single star point."
- note added: "HEADER_PINS — Test/Probe Access Breaks out stacking connector signals (J25–J28) to accessible pins for bench testing, mirroring each board's header pinout (3.3V, GND, GPIO, comms lines) without altering the signal path — lets you probe inter-board signals without disassembling the stack."
- note added: "OUTPUT — Actuation Breaks out GPIO to ESC, servo, and light headers (5V rail, per-channel pull resistors), routing Control's commands to motors/actuators to actually move the vehicle."
- note added: "POWER — Energy management Takes battery input (XT30, 4S2P pack) with surge/reverse protection, regulates to 3.3V, 5V, and 12V via buck converters, plus a boosted VPiezo rail (TPS55340) for the transducer. Includes voltage-divider power monitoring, status LEDs, and supplies power-good signals to the rest of the stack."
- note added: "SENSOR — Motion & environmental sensing I2C cluster: two IMUs (ASM330LHHXTR, LSM6DSO32TR), a magnetometer(MMC5603NJ), and a depth/pressure sensor (MS583730BA01-50). Shares one I2C bus with interrupt lines back to Control, which it feeds with orientation/environmental data."
- note added: "SYSTEM OVERVIEW ASTRELIS NAV (SWARM PCB) is the electronics stack for an autonomous underwater vehicle (AUV) intended to operate as part of a swarm. It senses its own orientation, motion, and depth (Sensor board), processes this data and runs navigation/control logic (Control board), communicates with other units or a base station acoustically via an underwater piezo transducer (TX/RX board), dri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"
- note added: "Splitting SWARM into five functional boards (Control, Power, Sensor, TX/RX, Output) stacked via headers — rather than one monolithic board or fully separate, individually-housed boards — balances modularity with integration: Noise isolation - Power (switching regulators) and TX/RX (sensitive RX analog, H-bridge) are separated from Sensor/Control, with isolated GND domains joined only at the stack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"
- note added: "TX/RX — Acoustic communication Two half-bridge MOSFET drivers (UCC27211) form an H-bridge driving the piezo transducer to transmit, with a precharge sequence at power-up. On receive, a preamp/instrumentation amp (INA823) and bandpass filter (20–30kHz, for FSK) feed a comparator; a T/R switch (ADG7421) isolates TX/RX paths, and an INA240 senses H-bridge current."
- note removed: "GND DOMAIN ARCHITECTURE Each subsystem has an isolated GND domain: GND_POWER, GND_CONTROL, GND_SENSOR, GND_TXRX, GND_HEADER. These domains are connected through the stacking connector pins (J25-J28). No single star point."
- moved on the sheet: J25, J26, J27, J28
