File: SWARM_PCB_Rev_2/SWARM_PCB_Rev_2.kicad_pcb (KiCad board)
At the start: 2 copper layers, 81.6 x 156.5 mm, 247 parts, among them J10 Conn_02x25_Odd_Even, J11 Conn_02x25_Odd_Even, J12 Conn_02x25_Odd_Even, J18 Conn_02x25_Odd_Even, J19 Conn_02x25_Odd_Even, J2 Conn_02x25_Odd_Even, J20 Conn_02x25_Odd_Even, J22 Conn_02x25_Odd_Even, J23 Conn_02x25_Odd_Even, J24 Conn_02x25_Odd_Even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

Commit message: Trace Tuning
Parts:
- moved dL2 0.35 mm to (52.5, 99.2)
Routing:
- net /TX_RX/RX_P: track 21.8 -> 18.0 mm, vias 0 -> 2
- net /TX_RX/Piezo_N: track 46.7 -> 50.0 mm
- net +3.3V_TXRX: track 102.7 -> 104.3 mm
- net /CONTROL/USB_D-: track 22.7 -> 23.9 mm
- net /SENSOR/SDA: track 72.8 -> 72.0 mm
- net GND_TXRX: vias 190 -> 223
- net GND_SENSOR: vias 227 -> 245
- net GND_CONTROL: vias 343 -> 342
