File: SWARM_PCB_Rev_2/SWARM_PCB_Rev_2.kicad_pcb (KiCad board)
At the start: 2 copper layers, 81.6 x 156.5 mm, 247 parts, among them J10 Conn_02x25_Odd_Even, J11 Conn_02x25_Odd_Even, J12 Conn_02x25_Odd_Even, J18 Conn_02x25_Odd_Even, J19 Conn_02x25_Odd_Even, J2 Conn_02x25_Odd_Even, J20 Conn_02x25_Odd_Even, J22 Conn_02x25_Odd_Even, J23 Conn_02x25_Odd_Even, J24 Conn_02x25_Odd_Even, J25 Conn_01x12_Pin, J26 Conn_01x12_Pin, J27 Conn_01x12_Pin, J28 Conn_01x13_Pin, J3 Conn_02x25_Odd_Even, J4 Conn_02x25_Odd_Even, J6 Conn_02x25_Odd_Even, J7 Conn_02x25_Odd_Even, J8 Conn_02x25_Odd_Even

Commit message: Design review fixes: feedback resistor, SWCLK, LED MPNs, GND annotation
- POWER: correct bR10 feedback resistor 187k→255k so TPS55340RTER
  (Vref=0.9V) sets VPiezo to 23.85V (~24V target)
- POWER: assign MPNs for bD2 (green), bD3/bD4 (blue) JE2835 LEDs
- CONTROL: add 33Ω series resistor aR18 on SWCLK near debug header aJ4
- CONTROL: assign MPNs for aD1 (purple) and aD2 (RGB) LEDs
- Top schematic: document isolated GND domain architecture (H3)
- PCB layout, sub-sheet, and SPICE updates

Co-Authored-By: Claude Sonnet 4.6 <noreply@anthropic.com>
Parts:
- added aR18: 33, Resistor_SMD:R_0603_1608Metric, F.Cu at (28.5, 66.5)
- bR10: value 187k -> 255k
- dC9: value 47u -> 10u; footprint Capacitor_SMD:C_0603_1608Metric -> Capacitor_SMD:C_1210_3225Metric
- moved dC9 0.74 mm to (27.5, 106.0)
Connections:
- JP1 pad 1: /CONTROL/SWCLK_P -> Net-(JP1-A)
Routing:
- net Net-(JP1-A): track 0.00 -> 5.47 mm
- net /CONTROL/SWCLK_P: track 14.0 -> 9.22 mm
- net /TX_RX/RX_N: track 15.7 -> 18.6 mm
- net /CONTROL/SWDIO: track 32.9 -> 34.6 mm
- net GND_TXRX: vias 223 -> 221
- net GND_CONTROL: vias 342 -> 341
