File: SWARM_PCB_Rev_2/SWARM_PCB_Rev_2.kicad_pcb (KiCad board)
At the start: 2 copper layers, 85.2 x 180.4 mm, 319 parts, among them J1 Conn_02x25_Odd_Even, J10 Conn_02x25_Odd_Even, J11 Conn_02x25_Odd_Even, J12 Conn_02x25_Odd_Even, J17 Conn_02x25_Odd_Even, J18 Conn_02x25_Odd_Even, J19 Conn_02x25_Odd_Even, J2 Conn_02x25_Odd_Even, J20 Conn_02x25_Odd_Even, J21 Conn_02x25_Odd_Even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

Commit message: Revert "to delete"
This reverts commit 543c70bcba01ecf78262208d4f10808184dfb0ad.
Routing:
- net GND_TXRX: vias 222 -> 223
