File: SWARM_PCB_Rev_2/HEADER_PINS.kicad_sch (KiCad schematic)
At the start: 4 parts, among them J2 Conn_02x25_Odd_Even, J3 Conn_02x25_Odd_Even, J4 Conn_02x25_Odd_Even

Commit message: Add MPNs to BOM and apply PCB DFM fixes for JLCPCB
Schematic: added MPN and Manufacturer properties to 205 references
across all sub-sheets (Murata/Yageo/TI/ST/Hirose/JST etc.).
Fixed dU7 description to match INA823DR (not INA828).

PCB: added via tenting (1540 vias), removed stale auto-placement-area
keepout zones (4 zones), increased annular rings on 482 undersized vias
(0.05mm -> 0.1mm), added 6 fiducial markers (3x F.Cu + 3x B.Cu).

Co-Authored-By: Claude Sonnet 4.6 <noreply@anthropic.com>
Parts:
- J2, J3, J4: MPN (none) -> DF40C-50DP-0.4V(51); Manufacturer (none) -> Hirose
Changed lines of the file:
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@@
+			)
+		)
+		(property "Manufacturer" "Hirose" (at 0 0 0)
+			(effects
+				(font
+					(size 1.27 1.27)
+				)
+				(hide yes)
+			)
+		)
+		(property "MPN" "DF40C-50DP-0.4V(51)" (at 0 0 0)
+			(effects
+				(font
+					(size 1.27 1.27)
+				)
+				(hide yes)
 			)
 		)
@@
 			)
 		)
+		(property "Manufacturer" "Hirose" (at 0 0 0)
+			(effects
+				(font
+					(size 1.27 1.27)
+				)
+				(hide yes)
+			)
+		)
+		(property "MPN" "DF40C-50DP-0.4V(51)" (at 0 0 0)
+			(effects
+				(font
+					(size 1.27 1.27)
+				)
+				(hide yes)
+			)
+		)
 		(pin "1"
 		)
@@
 			)
 		)
+		(property "Manufacturer" "Hirose" (at 0 0 0)
+			(effects
+				(font
+					(size 1.27 1.27)
+				)
+				(hide yes)
+			)
+		)
+		(property "MPN" "DF40C-50DP-0.4V(51)" (at 0 0 0)
+			(effects
+				(font
+					(size 1.27 1.27)
+				)
+				(hide yes)
+			)
+		)

Commit message: Fix T10/H1: swap dU1+dU2 VDD/VSS supply nets; populate J1 Value; close S4
T10 (Critical): UCC27211D dU1 and dU2 had VDD (pin 1) wired to GND_TXRX and
VSS (pin 7) wired to 12V_TXRX — completely inverted, would destroy chips at
power-on. Fixed by swapping lib_id and Value on four power symbols in
TX_RX.kicad_sch: VDD now on 12V_TXRX, VSS on GND_TXRX.

H1: J1 Value field was empty in HEADER_PINS.kicad_sch; set to
"Conn_02x25_Odd_Even" to match J2–J4.

S4: cU2 VDD_IO confirmed on +3.3V_SENSOR; INT1/INT2 wired separately —
no issue found, closed as confirmed-good.

Co-Authored-By: Claude Sonnet 4.6 <noreply@anthropic.com>
Parts:
- J1: value (none) -> Conn_02x25_Odd_Even
Changed lines of the file:
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@@
 			)
 		)
-		(property "Value" ""
+		(property "Value" "Conn_02x25_Odd_Even"
 			(at 38.1 24.13 0)
 			(hide yes)
