File: SWARM_PCB_Rev_2/HEADER_PINS.kicad_sch (KiCad schematic)
At the start: 4 parts, among them J1 Conn_02x25_Odd_Even, J2 Conn_02x25_Odd_Even, J3 Conn_02x25_Odd_Even, J4 Conn_02x25_Odd_Even

Commit message: Updated Via size to 0.25mm and ReExported Files
Parts:
- J2, J3, J4: Manufacturer Hirose -> (none)
Changed lines of the file:
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@@
-			)
-		)
-		(property "Manufacturer" "Hirose"
-			(at 0 0 0)
-			(hide yes)
-			(show_name no)
-			(do_not_autoplace no)
-			(effects
-				(font
-					(size 1.27 1.27)
-				)
 			)
 		)
@@
 			)
 		)
-		(property "Manufacturer" "Hirose"
-			(at 0 0 0)
-			(hide yes)
-			(show_name no)
-			(do_not_autoplace no)
-			(effects
-				(font
-					(size 1.27 1.27)
-				)
-			)
-		)
 		(property "MPN" "DF40C-50DP-0.4V(51)"
 			(at 0 0 0)
@@
 			(hide yes)
 			(show_name no)
-			(do_not_autoplace no)
-			(effects
-				(font
-					(size 1.27 1.27)
-				)
-			)
-		)
-		(property "Manufacturer" "Hirose"
-			(at 0 0 0)
-			(hide yes)
-			(show_name no)
