File: SWARM_PCB_Rev_2/TX_RX.kicad_sch (KiCad schematic)
At the start: 84 parts

Commit message: Add MPNs to BOM and apply PCB DFM fixes for JLCPCB
Schematic: added MPN and Manufacturer properties to 205 references
across all sub-sheets (Murata/Yageo/TI/ST/Hirose/JST etc.).
Fixed dU7 description to match INA823DR (not INA828).

PCB: added via tenting (1540 vias), removed stale auto-placement-area
keepout zones (4 zones), increased annular rings on 482 undersized vias
(0.05mm -> 0.1mm), added 6 fiducial markers (3x F.Cu + 3x B.Cu).

Co-Authored-By: Claude Sonnet 4.6 <noreply@anthropic.com>
Parts:
- dC1, dC16, dC2, dC29, dC3, dC30, dC4: MPN (none) -> GRM1885C1H102JA01D; Manufacturer (none) -> Murata
- dC10, dC12, dC13, dC15, dC17, dC18, dC19, dC20, dC21, dC22, dC24, dC26, dC32, dC5, dC6: MPN (none) -> GRM188R71C104KA01D; Manufacturer (none) -> Murata
- dC11, dC14: MPN (none) -> GRM21BR61A105KA73L; Manufacturer (none) -> Murata
- dC23: MPN (none) -> GRM21BR61A106KE18L; Manufacturer (none) -> Murata
- dC25, dC31: MPN (none) -> GRM188R61A105KA61D; Manufacturer (none) -> Murata
- dC27, dC28: MPN (none) -> GRM188R71H103KA01D; Manufacturer (none) -> Murata
- dC7, dC8: MPN (none) -> GRM32ER61A106KA88L; Manufacturer (none) -> Murata
- dC9: MPN (none) -> CL10A476MQ8NRNC; Manufacturer (none) -> Samsung
- dJ1: MPN (none) -> B3B-XH-AM; Manufacturer (none) -> JST
- dJ2: MPN (none) -> B8B-PH-SM4-TB(LF)(SN); Manufacturer (none) -> JST
- dQ1, dQ2, dQ3, dQ4: MPN (none) -> IPD50N10S3L-16; Manufacturer (none) -> Infineon Technologies
- dR1, dR2, dR3, dR4: MPN (none) -> RC0603FR-0747KL; Manufacturer (none) -> Yageo
- dR10, dR15, dR16, dR21, dR9: MPN (none) -> RC0603FR-0710RL; Manufacturer (none) -> Yageo
- dR11, dR14, dR19, dR20, dR5, dR8: MPN (none) -> RC0603FR-07100KL; Manufacturer (none) -> Yageo
- dR12, dR13, dR25, dR26, dR6, dR7: MPN (none) -> RC0603FR-07100RL; Manufacturer (none) -> Yageo
- dR17: MPN (none) -> WSL2512R0200FEA; Manufacturer (none) -> Vishay
- dR18: MPN (none) -> RC0603FR-071KL; Manufacturer (none) -> Yageo
- dR22, dR23, dR24, dR27, dR28, dR34: MPN (none) -> RC0603FR-0710KL; Manufacturer (none) -> Yageo
- dR29: MPN (none) -> RC0603FR-075K1L; Manufacturer (none) -> Yageo
- dR30: MPN (none) -> RC0603FR-07121RL; Manufacturer (none) -> Yageo
- dR31: MPN (none) -> RC0603FR-07953RL; Manufacturer (none) -> Yageo
- dR32: MPN (none) -> RC0603FR-073K83L; Manufacturer (none) -> Yageo
- dR33: MPN (none) -> RC0603FR-075K9L; Manufacturer (none) -> Yageo
- dR35, dR36: MPN (none) -> RC0603FR-073K92L; Manufacturer (none) -> Yageo
- dU1, dU2: MPN (none) -> UCC27211D; Manufacturer (none) -> Texas Instruments
- dU3: MPN (none) -> INA240A2DR; Manufacturer (none) -> Texas Instruments
- dU4: MPN (none) -> TLV9101IDCKR; Manufacturer (none) -> Texas Instruments
- dU5: MPN (none) -> ADG7421FBCPZ-RL7; Manufacturer (none) -> Analog Devices
- dU7: MPN (none) -> INA823DR; Manufacturer (none) -> Texas Instruments
- dU8: MPN (none) -> OPA2322AIDGKR; Manufacturer (none) -> Texas Instruments

Commit message: Design review fixes: feedback resistor, SWCLK, LED MPNs, GND annotation
- POWER: correct bR10 feedback resistor 187k→255k so TPS55340RTER
  (Vref=0.9V) sets VPiezo to 23.85V (~24V target)
- POWER: assign MPNs for bD2 (green), bD3/bD4 (blue) JE2835 LEDs
- CONTROL: add 33Ω series resistor aR18 on SWCLK near debug header aJ4
- CONTROL: assign MPNs for aD1 (purple) and aD2 (RGB) LEDs
- Top schematic: document isolated GND domain architecture (H3)
- PCB layout, sub-sheet, and SPICE updates

Co-Authored-By: Claude Sonnet 4.6 <noreply@anthropic.com>
Parts:
- dC7, dC8: MPN GRM32ER61A106KA88L -> GRM32ER71H106KA12
- dC9: value 47u -> 10u; footprint Capacitor_SMD:C_0603_1608Metric -> Capacitor_SMD:C_1210_3225Metric; MPN CL10A476MQ8NRNC -> GRM32ER71H106KA12; Manufacturer Samsung -> Murata
- dU7: MP INA828IDR -> INA823DR

Commit message: Design review fixes: cap voltage ratings, MPN corrections, FET symbol
- POWER: upgrade 17x MLCC MPNs to correct voltage ratings (6.3V/10V caps
  on 12–24V rails replaced with 25V/50V Murata GRM equivalents)
- POWER: fix bR10 MPN to RC0603FR-07255KL (was 187k part, value is 255k)
- CONTROL: fix aR18 MPN to RC0603FR-0733RL (was 10k part, value is 33R)
- TX_RX: replace IPD50R3K0CE lib symbol with Device:MOSFET_N for dQ1-dQ4
- TX_RX: mark dL1/dL2 value as TBD (piezo matching, pending characterisation)
- DESIGN_REVIEW: full review update with all findings by severity

Co-Authored-By: Claude Sonnet 4.6 <noreply@anthropic.com>
Parts:
- dL1, dL2: value (none) -> TBD
- dQ1, dQ2, dQ3, dQ4: symbol Transistor_FET:IPD50R3K0CE -> Device:MOSFET_N
Changed lines of the file:
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@@
 	)
 	(symbol
-		(lib_id "Transistor_FET:IPD50R3K0CE")
+		(lib_id "Device:MOSFET_N")
 		(at 44.45 38.1 0)
 		(unit 1)
@@
 	)
 	(symbol
-		(lib_id "Transistor_FET:IPD50R3K0CE")
+		(lib_id "Device:MOSFET_N")
 		(at 59.69 38.1 0)
 		(mirror y)
@@
 	)
 	(symbol
-		(lib_id "Transistor_FET:IPD50R3K0CE")
+		(lib_id "Device:MOSFET_N")
 		(at 59.69 25.4 0)
 		(mirror y)
@@
 	)
 	(symbol
-		(lib_id "Transistor_FET:IPD50R3K0CE")
+		(lib_id "Device:MOSFET_N")
 		(at 44.45 25.4 0)
 		(unit 1)
@@
 			)
 		)
-		(property "Value" ""
+		(property "Value" "TBD"
 			(at 209.55 72.136 90)
 			(show_name no)
@@
 			)
 		)
-		(property "Value" ""
+		(property "Value" "TBD"
 			(at 209.55 61.976 90)
 			(show_name no)

Commit message: Fix dU7 symbol: rename INA828IDR to INA823DR
INA823 and INA828 are pin-compatible (identical SOIC-8 pinout).
Renamed embedded lib symbol, sub-symbols, Value, MP, and lib_id
throughout TX_RX.kicad_sch. No connectivity changes required.

Co-Authored-By: Claude Sonnet 4.6 <noreply@anthropic.com>
Parts:
- dU7: symbol SWARM_Library:INA828IDR -> SWARM_Library:INA823DR; Check_prices https://www.snapeda.com/parts/INA828IDR/Texas+Instruments/v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 -> https://www.snapeda.com/parts/INA823DR/Texas+Instruments/vi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; SnapEDA_Link https://www.snapeda.com/parts/INA828IDR/Texas+Instruments/v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 -> https://www.snapeda.com/parts/INA823DR/Texas+Instruments/vi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
Changed lines of the file:
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@@
 	)
 	(symbol
-		(lib_id "SWARM_Library:INA828IDR")
+		(lib_id "SWARM_Library:INA823DR")
 		(at 245.11 138.43 0)
 		(unit 1)
@@
 			)
 		)
-		(property "SnapEDA_Link" "https://www.snapeda.com/parts/INA828IDR/Texas+Instruments/view-part/?ref=snap"
+		(property "SnapEDA_Link" "https://www.snapeda.com/parts/INA823DR/Texas+Instruments/view-part/?ref=snap"
 			(at 245.11 138.43 0)
 			(hide yes)
@@
 			)
 		)
-		(property "Check_prices" "https://www.snapeda.com/parts/INA828IDR/Texas+Instruments/view-part/?ref=eda"
+		(property "Check_prices" "https://www.snapeda.com/parts/INA823DR/Texas+Instruments/view-part/?ref=eda"
 			(at 245.11 138.43 0)
 			(hide yes)

Commit message: Fix T10/H1: swap dU1+dU2 VDD/VSS supply nets; populate J1 Value; close S4
T10 (Critical): UCC27211D dU1 and dU2 had VDD (pin 1) wired to GND_TXRX and
VSS (pin 7) wired to 12V_TXRX — completely inverted, would destroy chips at
power-on. Fixed by swapping lib_id and Value on four power symbols in
TX_RX.kicad_sch: VDD now on 12V_TXRX, VSS on GND_TXRX.

H1: J1 Value field was empty in HEADER_PINS.kicad_sch; set to
"Conn_02x25_Odd_Even" to match J2–J4.

S4: cU2 VDD_IO confirmed on +3.3V_SENSOR; INT1/INT2 wired separately —
no issue found, closed as confirmed-good.

Co-Authored-By: Claude Sonnet 4.6 <noreply@anthropic.com>
Connections:
- net 12V_TXRX: now also dU1.7 (VSS), dU2.7 (VSS); no longer dU1.1 (VDD), dU2.1 (VDD)
- net GND_TXRX: now also dU1.1 (VDD), dU2.1 (VDD); no longer dU1.7 (VSS), dU2.7 (VSS)
Changed lines of the file:
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@@
 	)
 	(symbol
-		(lib_id "power:+3.3V")
+		(lib_id "power:GND")
 		(at 68.58 100.33 0)
 		(unit 1)
@@
 			)
 		)
-		(property "Value" "12V_TXRX"
+		(property "Value" "GND_TXRX"
 			(at 68.58 97.028 0)
 			(show_name no)
@@
 	)
 	(symbol
-		(lib_id "power:GND")
+		(lib_id "power:+3.3V")
 		(at 68.58 83.82 0)
 		(unit 1)
@@
 			)
 		)
-		(property "Value" "GND_TXRX"
+		(property "Value" "12V_TXRX"
 			(at 68.58 87.376 0)
 			(show_name no)
@@
 	)
 	(symbol
-		(lib_id "power:GND")
+		(lib_id "power:+3.3V")
 		(at 68.58 124.46 0)
 		(unit 1)
@@
 			)
 		)
-		(property "Value" "GND_TXRX"
+		(property "Value" "12V_TXRX"
 			(at 68.58 128.016 0)
 			(show_name no)
@@
 	)
 	(symbol
-		(lib_id "power:+3.3V")
+		(lib_id "power:GND")
 		(at 68.58 59.69 0)
 		(unit 1)
@@
 			)
 		)
-		(property "Value" "12V_TXRX"
+		(property "Value" "GND_TXRX"
 			(at 68.58 56.388 0)
 			(show_name no)
