File: SWARM_PCB_Rev_2/TX_RX.kicad_sch (KiCad schematic)
At the start: 84 parts

Commit message: Fixed some small errors and added the Output board
Connections:
- net 12V_TXRX: now also dU1.1 (VDD), dU2.1 (VDD); no longer dU1.7 (VSS), dU2.7 (VSS)
- net GND_TXRX: now also dU1.7 (VSS), dU2.7 (VSS); no longer dU1.1 (VDD), dU2.1 (VDD)
