File: SWARM_PCB_Rev_2/TX_RX.kicad_sch (KiCad schematic)
At the start: 86 parts

Commit message: Resolved all DRC and ERC errors
Parts:
- dD1, dD2: MPN SS14-E3/61T -> (none); Manufacturer Vishay -> (none)
- dQ1, dQ2, dQ3, dQ4: symbol Device:MOSFET_N -> Simulation_SPICE:NMOS
- dU7: symbol SWARM_Library:INA823DR -> SWARM_Library:INA828IDR; Check_prices https://www.snapeda.com/parts/INA823DR/Texas+Instruments/vi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 -> https://www.snapeda.com/parts/INA828IDR/Texas+Instruments/v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; MP INA823DR -> INA828IDR; SnapEDA_Link https://www.snapeda.com/parts/INA823DR/Texas+Instruments/vi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 -> https://www.snapeda.com/parts/INA828IDR/Texas+Instruments/v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
Connections:
- net HO_A: now also dQ1.2 (G); no longer dQ1.1 (G)
- net HO_B: now also dQ3.2 (G); no longer dQ3.1 (G)
- net H_A: now also dQ2.1 (D); no longer dQ2.2 (D)
- net H_B: now also dQ4.1 (D); no longer dQ4.2 (D)
- net LO_A: now also dQ2.2 (G); no longer dQ2.1 (G)
- net LO_B: now also dQ4.2 (G); no longer dQ4.1 (G)
- net VPiezo_TXRX: now also dQ1.1 (D), dQ3.1 (D); no longer dQ1.2 (D), dQ3.2 (D)
Other:
- moved on the sheet: dC13, dC14, dC15, dC19, dC20, dC21, dC22, dC23, dC24, dC27, dC28, dC29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
