File: SWARM_PCB_Rev_2/POWER.kicad_sch (KiCad schematic)
At the start: 70 parts

Commit message: Design review fixes: P7/P8/C10/C11/T4 + MPN audit
- P7: bR3 36k→4.3k, bR4 82k→4.3k (blue LEDs now 2.05mA each)
- P8: bD1 lib_id Diode:SS34→Device:D_TVS; embed D_TVS lib_symbol in POWER.kicad_sch
- C10: aR19 33Ω (RC0603FR-0733RL) added on SWO line (user-placed)
- C11: aFB1 footprint Resistor_SMD:R_0603_1608Metric→Inductor_SMD:L_0603_1608Metric
- T4: dD1/dD2 SS14-E3/61T bootstrap Schottky diodes added on HB_A/HB_B; MPN set
- BOM: MPNs added to J25–J28 (Samtec SSQ), aJ1/aJ4 (Harwin M50)
- DESIGN_REVIEW.md: close T4, T8/T9, P7, P8, C10, C11, H2, dC9, bL1/bL2 items

Co-Authored-By: Claude Sonnet 4.6 <noreply@anthropic.com>
Parts:
- bC1: MPN GRM21BR61E225KA73L -> GRM21BR71H225KA12L
- bC14, bC21, bC26, bC4: MPN GRM21BR61E106KA73L -> GRM21BR71H106KA73L
Changed lines of the file:
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@@
 			)
 		)
-		(property "MPN" "GRM21BR61E106KA73L"
+		(property "MPN" "GRM21BR71H106KA73L"
 			(at 0 0 0)
 			(hide yes)
@@
 			)
 		)
-		(property "MPN" "GRM21BR61E106KA73L"
+		(property "MPN" "GRM21BR71H106KA73L"
 			(at 0 125.73 0)
 			(hide yes)
@@
 			)
 		)
-		(property "MPN" "GRM21BR61E106KA73L"
+		(property "MPN" "GRM21BR71H106KA73L"
 			(at 0 0 0)
 			(hide yes)
@@
 			)
 		)
-		(property "MPN" "GRM21BR61E225KA73L"
+		(property "MPN" "GRM21BR71H225KA12L"
 			(at 7.62 0 0)
 			(hide yes)
@@
 			)
 		)
-		(property "MPN" "GRM21BR61E106KA73L"
+		(property "MPN" "GRM21BR71H106KA73L"
 			(at 0 0 0)
 			(hide yes)
