File: SWARM_PCB_Rev_2/POWER.kicad_sch (KiCad schematic)
At the start: 70 parts

Commit message: Resolved all DRC and ERC errors
Parts:
- bU3: Availability (none) -> In Stock; Package (none) -> WQFN-16 Texas Instruments; Price (none) -> None
Other:
- moved on the sheet: bC21, bC22, bC23, bC24, bC25, bC26, bC27, bC28, bC29, bC30, bC31, bC32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

Commit message: Updated Via size to 0.25mm and ReExported Files
Parts:
- bC1, bC10, bC11, bC12, bC13, bC14, bC15, bC16, bC17, bC18, bC19, bC2, bC20, bC21, bC22, bC23, bC24, bC25, bC26, bC27, bC28, bC29, bC3, bC30, bC31, bC32, bC33, bC4, bC5, bC6, bC7, bC8, bC9: Manufacturer Murata -> (none)
- bD1, bD5: Manufacturer Vishay -> (none)
- bF1: Manufacturer Littelfuse -> (none)
- bJ1: Manufacturer Amass -> (none)
- bJ2: Manufacturer JST -> (none)
- bL1, bL2, bL4: Manufacturer Würth Elektronik -> (none)
- bL3: Manufacturer Panasonic -> (none)
- bR1, bR10, bR11, bR12, bR13, bR14, bR15, bR16, bR17, bR18, bR19, bR2, bR3, bR4, bR5, bR6, bR7, bR8, bR9: Manufacturer Yageo -> (none)
- bU1, bU2, bU4: Manufacturer Texas Instruments -> (none)
- bU3: Availability In Stock -> (none); Manufacturer Texas Instruments -> (none); Package WQFN-16 Texas Instruments -> (none); Price None -> (none)

Commit message: Cleaned up Schematic and Exported
Other:
- note added: "PG_3.3V → PB6 — digital, open-drain PG pin (pulled up via R6). LOW = 3.3V rail fault. PG_5V → PA10 — digital, open-drain PG pin (pulled up via R16). LOW = 5V rail fault. PG_12V → PB12 — digital, open-drain PG pin (pulled up via R9). LOW = 12V rail fault. PG_VPiezo → PB1 (ADC1_IN9) — analog, R11/R13 voltage divider sampling VPiezo rail. No digital flag — fault = ADC reading outside expected range."
Changed lines of the file:
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@@
+		)
+	)
+	(text "PG_3.3V → PB6 — digital, open-drain PG pin (pulled up via R6). LOW = 3.3V rail fault.\n\nPG_5V → PA10 — digital, open-drain PG pin (pulled up via R16). LOW = 5V rail fault.\n\nPG_12V → PB12 — digital, open-drain PG pin (pulled up via R9). LOW = 12V rail fault.\n\nPG_VPiezo → PB1 (ADC1_IN9) — analog, R11/R13 voltage divider sampling VPiezo rail. \nNo digital flag — fault = ADC reading outside expected range."
+		(exclude_from_sim no)
+		(at 134.366 138.684 0)
+		(effects
+			(font
+				(size 2.032 2.032)
+			)
+			(justify left)
 		)
 	)
