File: SWARM_PCB_Rev_2/OUTPUT.kicad_sch (KiCad schematic)
At the start: 29 parts

Commit message: Resolved all DRC and ERC errors
Other:
- title: (none) -> OUTPUT
Changed lines of the file:
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@@
 	(paper "A4")
 	(title_block
-		(date "2026-05-27")
+		(title "OUTPUT")
+		(date "2026-06-19")
+		(rev "1")
 		(company "ASTRELIS NAV")
 		(comment 1 "By SAMANTHA CHONG")
